File: BMS_Testing.kicad_sch (KiCad schematic)
At the start: 101 parts, among them J1 Voltage Taps, J2 Thermistor 1, J3 Thermistor 2, J4 Thermistor 2, Q1 NPN, Q2 CSD19532Q5B, Q3 CSD19532Q5B, U1 BQ7695202PFB

Commit message: Add transient BMS simulation models
Add MOSFET and constant-current load models, configure schematic simulation properties and transient analysis, and include a simulation result.
Connections:
- net 0: no longer C29.2, I1.2, R18.2, R20.1
- net at R9.2, U1.8 (VC8): now also C10.2, C9.1
- net at R33.1: now also U1.43 (DSG); no longer D1.2 (A)
- net CD: now reaches Q2.5 (D), Q3.5 (D)
- net CD: now also D1.2 (A)
- new net BUS-: C29.2, I1.2, R18.2, R20.1
Other:
- note added: ".options rshunt=1e12 method=gear reltol=1e-3"
Changed lines of the file:
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@@
 	)
 	(junction
+		(at 105.41 138.43)
+		(diameter 0)
+		(color 0 0 0 0)
+	)
+	(label "CD"
+		(at 289.56 142.24 0)
+		(effects
+			(font
+				(size 1.27 1.27)
+			)
+			(justify left bottom)
+		)
+	)
+	(label "CD"
+		(at 279.4 45.72 0)
+		(effects
+			(font
+				(size 1.27 1.27)
+			)
+			(justify left bottom)
+		)
+	)
+	(text ".options rshunt=1e12 method=gear reltol=1e-3"
+		(exclude_from_sim no)
+		(at 25.4 259.08 0)
+		(effects
+			(font
+				(size 1.27 1.27)
+			)
+			(justify left bottom)
+		)
+	)
+	(junction
 		(at 62.23 224.79)
 		(diameter 0)
@@
 	(wire
 		(pts
-			(xy 289.56 81.28) (xy 289.56 142.24)
+			(xy 289.56 81.28) (xy 289.56 125.73)
 		)
 		(stroke
@@
 		(unit 1)
 		(body_style 1)
-		(exclude_from_sim no)
+		(exclude_from_sim yes)
 		(in_bom yes)
 		(on_board yes)
@@
 		(unit 1)
 		(body_style 1)
-		(exclude_from_sim no)
+		(exclude_from_sim yes)
 		(in_bom yes)
 		(on_board yes)
@@
 			)
 		)
-		(property "Sim.Pins" "1=+ 2=-"
+		(property "Sim.Pins" "1=P 2=N"
 			(at 386.08 119.38 0)
 			(hide yes)
@@
 			)
 		)
-		(property "Sim.Type" "DC"
+		(property "Sim.Device" "SUBCKT"
 			(at 386.08 119.38 0)
 			(hide yes)
@@
 			)
 		)
-		(property "Sim.Device" "I"
+		(property "Sim.Library" "sim_loads.lib"
+			(at 386.08 119.38 0)
+			(hide yes)
+			(show_name no)
+			(do_not_autoplace no)
+			(effects
+				(font
+					(size 1.27 1.27)
+				)
+			)
+		)
+		(property "Sim.Name" "LOAD_CC"
+			(at 386.08 119.38 0)
+			(hide yes)
+			(show_name no)
+			(do_not_autoplace no)
+			(effects
+				(font
+					(size 1.27 1.27)
+				)
+			)
+		)
+		(property "Sim.Params" "I=50 TON=0.4 TRISE=1m"
 			(at 386.08 119.38 0)
 			(hide yes)
@@
 			)
 		)
-		(property "Sim.Device" "NMOS"
+		(property "Sim.Device" "SUBCKT"
 			(at 269.24 48.26 0)
 			(hide yes)
@@
 			)
 		)
-		(property "Sim.Type" "VDMOS"
+		(property "Sim.Pins" "1=S 4=G 5=D"
 			(at 269.24 48.26 0)
 			(hide yes)
@@
 			)
 		)
-		(property "Sim.Pins" "1=D 2=G 3=S 4=<TJ> 5=<TCASE>"
+		(property "Sim.Library" "csd19532q5b.lib"
+			(at 269.24 48.26 0)
+			(hide yes)
+			(show_name no)
+			(do_not_autoplace no)
+			(effects
+				(font
+					(size 1.27 1.27)
+				)
+			)
+		)
+		(property "Sim.Name" "CSD19532Q5B"
 			(at 269.24 48.26 0)
 			(hide yes)
@@
 			)
 		)
+		(property "Sim.Device" "R"
+			(at 83.82 208.28 0)
+			(hide yes)
+			(show_name no)
+			(do_not_autoplace no)
+			(effects
+				(font
+					(size 1.27 1.27)
+				)
+			)
+		)
+		(property "Sim.Pins" "1=+ 2=-"
+			(at 83.82 208.28 0)
+			(hide yes)
+			(show_name no)
+			(do_not_autoplace no)
+			(effects
+				(font
+					(size 1.27 1.27)
+				)
+			)
+		)
+		(property "Sim.Params" "r=10u"
+			(at 83.82 208.28 0)
+			(hide yes)
+			(show_name no)
+			(do_not_autoplace no)
+			(effects
+				(font
+					(size 1.27 1.27)
+				)
+			)
+		)
 		(pin "1"
 		)
@@
 			)
 		)
-		(property "Value" "0"
+		(property "Value" "BUS-"
 			(at 161.29 229.108 0)
 			(show_name no)
@@
 			)
 		)
-		(property "Sim.Pins" "1=A 2=K"
+		(property "Sim.Pins" "1=K 2=A"
+			(at 335.28 142.24 0)
+			(hide yes)
+			(show_name no)
+			(do_not_autoplace no)
+			(effects
+				(font
+					(size 1.27 1.27)
+				)
+			)
+		)
+		(property "Sim.Params" "is=1u n=1.05 rs=50m cjo=150p bv=100 ibv=10u"
 			(at 335.28 142.24 0)
 			(hide yes)
@@
 		(unit 1)
 		(body_style 1)
-		(exclude_from_sim no)
+		(exclude_from_sim yes)
 		(in_bom yes)
 		(on_board yes)
@@
 		(unit 1)
 		(body_style 1)
-		(exclude_from_sim no)
+		(exclude_from_sim yes)
 		(in_bom yes)
 		(on_board yes)
@@
 			)
 		)
-		(property "Sim.Device" "NMOS"
+		(property "Sim.Device" "SUBCKT"
 			(at 289.56 48.26 0)
 			(hide yes)
@@
 			)
 		)
-		(property "Sim.Type" "VDMOS"
+		(property "Sim.Pins" "1=S 4=G 5=D"
 			(at 289.56 48.26 0)
 			(hide yes)
@@
 			)
 		)
-		(property "Sim.Pins" "1=D 2=G 3=S 4=<TJ> 5=<TCASE>"
+		(property "Sim.Library" "csd19532q5b.lib"
+			(at 289.56 48.26 0)
+			(hide yes)
+			(show_name no)
+			(do_not_autoplace no)
+			(effects
+				(font
+					(size 1.27 1.27)
+				)
+			)
+		)
+		(property "Sim.Name" "CSD19532Q5B"
 			(at 289.56 48.26 0)
 			(hide yes)
@@
 			)
 		)
-		(property "Sim.Pins" "1=A 2=K"
+		(property "Sim.Pins" "1=K 2=A"
+			(at 185.42 71.12 0)
+			(hide yes)
+			(show_name no)
+			(do_not_autoplace no)
+			(effects
+				(font
+					(size 1.27 1.27)
+				)
+			)
+		)
+		(property "Sim.Params" "is=1u n=1.05 rs=50m cjo=150p bv=100 ibv=10u"
 			(at 185.42 71.12 0)
 			(hide yes)
@@
 			)
 		)
+		(property "Sim.Params" "REG2_V=5"
+			(at 228.6 153.67 0)
+			(hide yes)
+			(show_name no)
+			(do_not_autoplace no)
+			(effects
+				(font
+					(size 1.27 1.27)
+				)
+			)
+		)
 		(pin "5"
 		)
@@
 			)
 		)
-		(property "Value" "0"
+		(property "Value" "BUS-"
 			(at 351.79 98.298 0)
 			(show_name no)
@@
 			)
 		)
-		(property "Sim.Pins" "1=A 2=K"
+		(property "Sim.Pins" "1=K 2=A"
+			(at 242.57 52.07 0)
+			(hide yes)
+			(show_name no)
+			(do_not_autoplace no)
+			(effects
+				(font
+					(size 1.27 1.27)
+				)
+			)
+		)
+		(property "Sim.Params" "is=1e-12 n=1.2 rs=5 bv=16 ibv=1m cjo=50p"
 			(at 242.57 52.07 0)
 			(hide yes)
@@
 			)
 		)
-		(property "Sim.Pins" "1=A 2=K"
+		(property "Sim.Pins" "1=K 2=A"
+			(at 312.42 52.07 0)
+			(hide yes)
+			(show_name no)
+			(do_not_autoplace no)
+			(effects
+				(font
+					(size 1.27 1.27)
+				)
+			)
+		)
+		(property "Sim.Params" "is=1e-12 n=1.2 rs=5 bv=16 ibv=1m cjo=50p"
 			(at 312.42 52.07 0)
 			(hide yes)
@@
 		(unit 1)
 		(body_style 1)
-		(exclude_from_sim no)
+		(exclude_from_sim yes)
 		(in_bom yes)
 		(on_board yes)
@@
 		(unit 1)
 		(body_style 1)
-		(exclude_from_sim no)
+		(exclude_from_sim yes)
 		(in_bom yes)
 		(on_board yes)
@@
 		(unit 1)
 		(body_style 1)
-		(exclude_from_sim no)
+		(exclude_from_sim yes)
 		(in_bom yes)
 		(on_board yes)
@@
 		(unit 1)
 		(body_style 1)
-		(exclude_from_sim no)
+		(exclude_from_sim yes)
 		(in_bom yes)
 		(on_board yes)

Commit message: Model thermal cell behavior and add probes
Add temperature- and SOC-dependent cell resistance, thermal modeling, and pack/BMS measurement probes. Update load and BQ76952 models for more robust simulations, configure a 45 A, 400 s run, and include its result.
Parts:
- added TP4: Ah out (true), symbol Connector:TestPoint
- added TP5: Ah out (BMS count), symbol Connector:TestPoint
- added TP6: SOC % (true), symbol Connector:TestPoint
- added TP7: SOC % (BMS est.), symbol Connector:TestPoint
- added TP8: Cell temp degC, symbol Connector:TestPoint
Connections:
- new net BMS_AH_OUT: TP5.1
- new net BMS_SOC: TP7.1
- new net PACK_AH_OUT: TP4.1
- new net PACK_SOC: TP6.1
- new net PACK_TEMP: TP8.1
Other:
- note added: "SIMULATION PROBES (sim only: not in BOM / not on PCB). In the simulator, click the wire to plot. 1 V = 1 Ah, 1 V = 1 %, 1 V = 1 degC. PACK_* = true values from the cell models (average over cells), BMS_* = BQ76952 coulomb counter"

Commit message: Add programmable loads and cell variation
Add profile-driven load modes, load telemetry probes, and per-cell variation/self-discharge parameters. Tune BMS protection defaults for the 16S1P Molicel P45B pack and include a simulation result.
Parts:
- added I2: 0, Package_TO_SOT_SMD:SOT-416, symbol Simulation_SPICE:IDC
- added TP10: Load power W, symbol Connector:TestPoint
- added TP11: Load energy Wh, symbol Connector:TestPoint
- added TP9: Load current A, symbol Connector:TestPoint
- I1: value 50 -> LOAD_PROFILE (see Sim.Params)
Connections:
- net 0: now also I2.1
- new net LOAD_CTRL: I2.2
- new net LOAD_I: TP9.1
- new net LOAD_P: TP10.1
- new net LOAD_WH: TP11.1
Other:
- note added: "LOAD PROFILE SOURCE (used when load I1 has PROF=2) Set I2 to any KiCad source type - PWL drive cycle, pulse, sine, random... Its value becomes the load set-point: A (MODE=0), W (1), ohm (2) or V (3)."

Commit message: Add BMS drive-cycle simulation dashboard
Configure a 1700-second demo cycle with BMS-aware load interlocking, balancing behavior, and simulated fault scenarios. Add probe signals and waveform traces for pack state, cell voltages, charge throughput, faults, FETs, and balancing.
Parts:
- added TP12: Pack voltage V, symbol Connector:TestPoint
- added TP13: BMS fault code, symbol Connector:TestPoint
- added TP14: ah dis x10, symbol Connector:TestPoint
- added TP15: ah chg x10, symbol Connector:TestPoint
- added TP16: bms ah dis x10, symbol Connector:TestPoint
- added TP17: bms ah chg x10, symbol Connector:TestPoint
- added TP18: cell max x10, symbol Connector:TestPoint
- added TP19: cell min x10, symbol Connector:TestPoint
- added TP20: cell spread mv, symbol Connector:TestPoint
- added TP21: bms fets, symbol Connector:TestPoint
- added TP22: bms balancing, symbol Connector:TestPoint
- I2: value 0 -> demo cycle (PWL)
Connections:
- new net AH_CHG_X10: TP15.1
- new net AH_DIS_X10: TP14.1
- new net BMS_AH_CHG_X10: TP17.1
- new net BMS_AH_DIS_X10: TP16.1
- new net BMS_BALANCING: TP22.1
- new net BMS_FAULT: TP13.1
- new net BMS_FETS: TP21.1
- new net CELL_MAX_X10: TP18.1
- new net CELL_MIN_X10: TP19.1
- new net CELL_SPREAD_MV: TP20.1
- new net PACK_V: TP12.1
Other:
- note added: ".save v(PACK_V) v(LOAD_I) v(LOAD_P) v(LOAD_WH) v(LOAD_CTRL) v(PACK_SOC) v(BMS_SOC) v(PACK_AH_OUT) v(BMS_AH_OUT) v(AH_DIS_X10) v(AH_CHG_X10) v(BMS_AH_DIS_X10) v(BMS_AH_CHG_X10) v(CELL_MAX_X10) v(CELL_MIN_X10) v(CELL_SPREAD_MV) v(PACK_TEMP) v(BMS_FAULT) v(BMS_FETS) v(BMS_BALANCING) v(BMS_DSG_OK) v(BMS_CHG_OK)"
- note added: "BMS_FAULT: 10 COV 20 CUV 30 OCC 40 OCD1-3 50 SCD 60 OT/UT 70 PF (0 = none) BMS_FETS: 10 = CHG FET on, +5 = DSG FET on (15 = both) BMS_BALANCING = cells selected *_X10 nets are scaled x10 to share the 0-100 axis: CELL_MAX_X10 42.5 = 4.25 V, AH_DIS_X10 12 = 1.2 Ah"
- note added: "DEFAULT SIMULATION - open the simulator and press Run (TRAN tab, 1700 s of pack time; a few minutes to compute). 16S Molicel P45B pack, cells start at ~30 % SOC with cell-to-cell deviations (BT1-BT16 Sim.Params). I2 plays this cycle into load I1: 0-300 s drive-cycle discharge 15/45/5 A -> weakest cell hits 2.53 V -> CUV trips, load interlock stops discharging 300-320 s rest, 320 s 13 A CC charge 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"
- note added: "LOAD PROFILE SOURCE I2 - drives load I1 (I1 has PROF=2) Default: the demo charge/discharge cycle as a PWL list (amps, + = discharge). Change it to any KiCad source type (PWL drive cycle, pulse, sine, random...). The value becomes I1's set-point: A (MODE=0), W (1), ohm (2) or V (3)."
- note added: "^ this .save keeps the run fast/small: only these signals are stored. To probe any other net, tick 'Save all voltages' in Sim Command settings."
- note removed: "LOAD PROFILE SOURCE (used when load I1 has PROF=2) Set I2 to any KiCad source type - PWL drive cycle, pulse, sine, random... Its value becomes the load set-point: A (MODE=0), W (1), ohm (2) or V (3)."
